File: hardware/schematics/PowerDeliveryBoard.sch (EAGLE design)
At the start: 18 parts

Commit message: added review comments
Other:
- note added: "The footprint for this is not the XT-60 connector that I assume we will be using. It needs to be correct so that when you layout the board and we fab it the connector will fit."
- note added: "The measuring point should be netted to the MCU whenever it is added. This would mess up the 3.3 rail and cause bad measurements."
- note added: "These reg footprints look closer but they don't have the no-go zone for them to be folded back, or the through hole to hold them on."
- note added: "This is redundant, board layout should be done in the board file."
Changed lines of the file:
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@@
 <text x="149.86" y="99.06" size="1.778" layer="91" grouprefs="POWERDELIVERYBOARD">5V Regulator</text>
 <text x="7.62" y="66.04" size="1.778" layer="91" grouprefs="POWERDELIVERYBOARD">Lipo Battery</text>
+<text x="-111.76" y="210.82" size="2.54" layer="91">The footprint for this is not the XT-60 connector that I assume we will
+ be using. It needs to be correct so that when you layout the board
+ and we fab it the connector will fit.</text>
+<text x="33.02" y="218.44" size="2.54" layer="91">These reg footprints look closer but they don't have the no-go zone for
+them to be folded back, or the through hole to hold them on.</text>
+<text x="132.08" y="157.48" size="1.778" layer="91">The measuring point should be netted to the MCU whenever it is
+ added. This would mess up the 3.3 rail and cause bad measurements.</text>
+<text x="55.88" y="121.92" size="2.54" layer="91">This is redundant, board layout should be done in the board file.</text>
 </plain>
 <instances>
@@
 </drawing>
 <compatibility>
+<note version="6.3" minversion="6.2.2" severity="warning">
+Since Version 6.2.2 text objects can contain more than one line,
+which will not be processed correctly with this version.
+</note>
 <note version="8.2" severity="warning">
 Since Version 8.2, EAGLE supports online libraries. The ids

Commit message: updated changes for power schematic
Parts:
- removed 3.3VREG, U$4: 5VREG, Power_Delivery_Board:5VREG
- removed C1, C2, C3, C4: (no value), rcl:C-EU025-024X044
- removed R: 10k, rcl:R-US_0204/2V
- removed R1: THERMISTOR-5, varistor:THERMISTOR-5
- removed U$1, U$5: LIPOBATT, Power_Delivery_Board:LIPOBATT
- removed U$2, U$3: 3VREG, Power_Delivery_Board:3VREG
- added IC1, IC2: 7812T, linear:7812T
- added J1: XT60-M, XT60-M:XT60-M
Connections:
- removed net 3.3V: C4.2, R1.1, U$2.VOUT
- net 0: now also IC1.GND, IC2.GND, J1.-; no longer 3.3VREG.GND, C1.2, C2.1, C3.2, C4.1, R.1, U$1.GND, U$2.GND, U$3.GND, U$4.GND, U$5.GND
- net VCC: now also IC1.VI, IC1.VO, IC2.VI, IC2.VO, J1.+; no longer 3.3VREG.VIN, 3.3VREG.VOUT, C1.1, C2.2, C3.1, R.2, R1.2, U$1.VCC, U$2.VIN, U$3.VIN, U$3.VOUT, U$4.VIN, U$4.VOUT, U$5.VCC
Other:
- note removed: "3.3V Regulator"
- note removed: "5V Regulator"
- note removed: "Lipo Battery"
- note removed: "The footprint for this is not the XT-60 connector that I assume we will be using. It needs to be correct so that when you layout the board and we fab it the connector will fit."
- note removed: "The measuring point should be netted to the MCU whenever it is added. This would mess up the 3.3 rail and cause bad measurements."
- note removed: "These reg footprints look closer but they don't have the no-go zone for them to be folded back, or the through hole to hold them on."
- note removed: "This is redundant, board layout should be done in the board file."
- moved on the sheet: C5, C6, C7, C8, R2, R3

Commit message: added review notes
Other:
- note added: "Although the package footprints were the same, the pinout for the regulators were different last year. If we are using the same 3v3 reg then we will have to account for that. Look at the datasheet of whatever regualtor we are getting to check the exact pinout"
- note added: "This resistor footprint looks small. Make sure we will be able to actually fit the resistors on the board"
Changed lines of the file:
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@@
 <sheet>
 <plain>
+<text x="53.34" y="43.18" size="1.778" layer="91">Although the package footprints were the same, the pinout for the
+regulators were different last year. If we are using the same 3v3 reg
+then we will have to account for that. Look at the datasheet of whatever
+regualtor we are getting to check the exact pinout</text>
+<text x="182.88" y="-7.62" size="1.778" layer="91">This resistor footprint looks small. Make sure we will be able to actually
+fit the resistors on the board</text>
 </plain>
 <instances>
@@
 </drawing>
 <compatibility>
+<note version="6.3" minversion="6.2.2" severity="warning">
+Since Version 6.2.2 text objects can contain more than one line,
+which will not be processed correctly with this version.
+</note>
 <note version="8.2" severity="warning">
 Since Version 8.2, EAGLE supports online libraries. The ids
